File: main.brd (EAGLE design)
At the start: 68.6 x 53.3 mm, 4 parts, among them J2 HDR-1X6, J5 HDR-2X8, J6 HDR-2X8, J7 HDR-2X6

Commit message: Add files via upload
Parts:
- added CN1: (no value), con-amp-mt6:MT6-8
- added F1: 1A, fuse:PICOFUSE
- added LD1, LD2: (no value), led:LD260
- added R1: 10K, rcl:0204/5
- added R2: 2.2K, rcl:0204/5
- added REG1: 5V, v-reg:78XXL
Connections:
- new net S$1: F1.1
- new net S$3: F1.2, LD1.K, LD2.A
- new net S$4: LD1.A, R1.2
- new net S$7: LD2.K, R2.2
- new net S$8: R1.1, R2.1, REG1.GND
Routing:
- net S$8: track 0.00 -> 55.6 mm
- net S$3: track 0.00 -> 40.9 mm
- net S$4: track 0.00 -> 16.8 mm
- net S$1: track 0.00 -> 8.77 mm
- net S$7: track 0.00 -> 4.07 mm
Other:
- board size 68.6 x 53.3 mm -> 112.4 x 53.3 mm
Changed lines of the file:
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@@
 <setting verticaltext="up"/>
 </settings>
-<grid distance="0.01" unitdist="inch" unit="inch" style="lines" multiple="1" display="yes" altdistance="0.025" altunitdist="inch" altunit="inch"/>
+<grid distance="0.025" unitdist="inch" unit="inch" style="lines" multiple="1" display="yes" altdistance="0.025" altunitdist="inch" altunit="inch"/>
 <layers>
 <layer number="1" name="Top" color="4" fill="1" visible="yes" active="yes"/>
@@
 <board>
 <plain>
-<wire x1="0" y1="0" x2="68.58" y2="0" width="0" layer="20"/>
-<wire x1="68.58" y1="0" x2="68.58" y2="53.34" width="0" layer="20"/>
-<wire x1="68.58" y1="53.34" x2="0" y2="53.34" width="0" layer="20"/>
-<wire x1="0" y1="53.34" x2="0" y2="0" width="0" layer="20"/>
+<wire x1="-37.455" y1="0" x2="74.93" y2="0" width="0" layer="20"/>
+<wire x1="74.93" y1="0" x2="74.93" y2="53.34" width="0" layer="20"/>
+<wire x1="74.93" y1="53.34" x2="-37.455" y2="53.34" width="0" layer="20"/>
+<wire x1="-37.455" y1="53.34" x2="-37.455" y2="0" width="0" layer="20"/>
 <wire x1="60.706" y1="45.212" x2="61.214" y2="45.72" width="0.2032" layer="21"/>
 <wire x1="61.214" y1="45.72" x2="61.722" y2="45.212" width="0.2032" layer="21"/>
@@
 <text x="33.528" y="4.318" size="1.016" layer="21" ratio="12" rot="R90">RESET</text>
 <text x="46.228" y="4.318" size="1.016" layer="21" ratio="12" rot="R90">VIN</text>
-<hole x="15.24" y="50.8" drill="3.2004"/>
-<hole x="66.04" y="35.56" drill="3.2004"/>
-<hole x="66.04" y="7.62" drill="3.2004"/>
+<circle x="-19.685" y="11.43" radius="1.27" width="0.4064" layer="20"/>
+<circle x="-19.685" y="41.91" radius="1.27" width="0.4064" layer="20"/>
+<circle x="71.755" y="41.91" radius="1.27" width="0.4064" layer="20"/>
+<circle x="71.755" y="10.16" radius="1.27" width="0.4064" layer="20"/>
+<dimension x1="74.93" y1="53.34" x2="-37.455" y2="53.34" x3="18.7375" y3="60.325" layer="20" dtype="horizontal"/>
 </plain>
 <attributes>
@@
 <attribute name="NAME" x="66.294" y="1.524" size="1.016" layer="25" rot="R90"/>
 </element>
+<element name="CN1" library="con-amp-mt6" package="MT6-8" value="" x="-29.21" y="10.16" rot="R90"/>
+<element name="F1" library="fuse" package="PICOFUSE" value="1A" x="-27.305" y="48.26"/>
+<element name="LD1" library="led" package="LD260" value="" x="-18.415" y="50.165"/>
+<element name="LD2" library="led" package="LD260" value="" x="-13.335" y="50.165" rot="R180"/>
+<element name="R1" library="rcl" package="0204/5" value="10K" x="-35.56" y="48.895" rot="R90"/>
+<element name="REG1" library="v-reg" package="78XXL" value="5V" x="-3.81" y="37.465"/>
+<element name="R2" library="rcl" package="0204/5" value="2.2K" x="-13.97" y="43.815" rot="R90"/>
 </elements>
 <signals>
@@
 <signal name="N$47">
 </signal>
+<signal name="S$1">
+<wire x1="-29.21" y1="40.64" x2="-29.21" y2="44.45" width="1.9304" layer="16"/>
+<wire x1="-29.21" y1="44.45" x2="-32.385" y2="48.26" width="1.9304" layer="16"/>
+<contactref element="F1" pad="1"/>
+</signal>
+<signal name="S$3">
+<contactref element="F1" pad="2"/>
+<contactref element="LD1" pad="K"/>
+<wire x1="-20.955" y1="46.99" x2="-17.78" y2="47.625" width="0.6096" layer="16"/>
+<wire x1="-17.78" y1="47.625" x2="-17.145" y2="48.26" width="0.6096" layer="16"/>
+<wire x1="-17.145" y1="48.26" x2="-17.145" y2="50.165" width="0.6096" layer="16"/>
+<wire x1="-22.225" y1="48.26" x2="-20.955" y2="46.99" width="1.9304" layer="16"/>
+<wire x1="-20.955" y1="46.99" x2="-17.78" y2="46.99" width="1.9304" layer="16"/>
+<wire x1="-17.78" y1="46.99" x2="-14.605" y2="43.815" width="1.9304" layer="16"/>
+<wire x1="-14.605" y1="43.815" x2="-13.97" y2="43.815" width="1.9304" layer="16"/>
+<wire x1="-13.97" y1="43.815" x2="-9.525" y2="43.815" width="1.9304" layer="16"/>
+<wire x1="-9.525" y1="43.815" x2="-6.35" y2="40.64" width="1.9304" layer="16"/>
+<wire x1="-6.35" y1="40.64" x2="-6.35" y2="33.02" width="1.9304" layer="16"/>
+<contactref element="LD2" pad="A"/>
+<wire x1="-13.97" y1="43.815" x2="-12.065" y2="43.815" width="0.6096" layer="16"/>
+<wire x1="-12.065" y1="43.815" x2="-12.065" y2="50.165" width="0.6096" layer="16"/>
+</signal>
+<signal name="S$4">
+<contactref element="LD1" pad="A"/>
+<wire x1="-19.685" y1="50.165" x2="-22.225" y2="52.07" width="0.6096" layer="16"/>
+<wire x1="-22.225" y1="52.07" x2="-34.925" y2="52.07" width="0.6096" layer="16"/>
+<contactref element="R1" pad="2"/>
+<wire x1="-34.925" y1="52.07" x2="-35.56" y2="51.435" width="0.6096" layer="16"/>
+</signal>
+<signal name="S$7">
+<contactref element="R2" pad="2"/>
+<contactref element="LD2" pad="K"/>
+<wire x1="-13.97" y1="46.355" x2="-14.605" y2="46.99" width="0.6096" layer="16"/>
+<wire x1="-14.605" y1="46.99" x2="-14.605" y2="50.165" width="0.6096" layer="16"/>
+</signal>
+<signal name="S$8">
+<contactref element="R2" pad="1"/>
+<wire x1="-13.97" y1="41.275" x2="-13.97" y2="39.37" width="0.6096" layer="16"/>
+<wire x1="-13.97" y1="39.37" x2="-17.145" y2="36.195" width="0.6096" layer="16"/>
+<contactref element="R1" pad="1"/>
+<wire x1="-35.56" y1="46.355" x2="-35.56" y2="39.37" width="0.6096" layer="16"/>
+<wire x1="-35.56" y1="39.37" x2="-32.385" y2="36.195" width="0.6096" layer="16"/>
+<wire x1="-32.385" y1="36.195" x2="-29.21" y2="36.195" width="0.6096" layer="16"/>
+<wire x1="-29.21" y1="36.195" x2="-18.415" y2="36.195" width="1.9304" layer="16"/>
+<wire x1="-18.415" y1="36.195" x2="-16.51" y2="36.195" width="1.9304" layer="16"/>
+<wire x1="-16.51" y1="36.195" x2="-8.89" y2="28.575" width="1.9304" layer="16"/>
+<wire x1="-8.89" y1="28.575" x2="-4.445" y2="28.575" width="1.9304" layer="16"/>
+<contactref element="REG1" pad="GND"/>
+<wire x1="-4.445" y1="28.575" x2="-3.81" y2="29.21" width="1.9304" layer="16"/>
+<wire x1="-3.81" y1="29.21" x2="-3.81" y2="33.655" width="1.9304" layer="16"/>
+<wire x1="-17.145" y1="36.195" x2="-18.415" y2="36.195" width="0.6096" layer="16"/>
+</signal>
 </signals>
